Commit message: add gz_launch, urdf fix for gz

File: description/drone_core.xacro (robot description, xacro)
@@ -1,62 +1,113 @@
 <?xml version="1.0"?>
 <robot xmlns:xacro="http://www.ros.org/wiki/xacro"  >
-    <material name="gray">
+      <xacro:include filename="inertial_macros.xacro"/>
+      <material name="gray">
         <color rgba="0.5 0.5 0.5 1.0"/>
-    </material>
-    <material name="white">
+      </material>
+      <material name="white">
         <color rgba="0.9 0.9 0.9 1.0"/>
-    </material>
-    <material name="red">
+      </material>
+      <material name="red">
         <color rgba="1.0 0 0 1.0"/>
-    </material>
-    <link name="base_link">
-       <visual>
-		 <origin xyz="0 0 0" rpy="0 0 0" />
-         <geometry>
-           <box size="0.4 0.2 0.04"/>
-         </geometry>
-         <material name="gray"/>
-       </visual>
-     </link>
-     <link name="FL">
-       <visual>
-		 <origin xyz="0 0 0.04" rpy="${pi/2} 0 0" />
-         <geometry>
+      </material>
+      <link name="base_link">
+        <visual>
+          <origin xyz="0 0 0" rpy="0 0 0" />
+          <geometry>
+            <box size="0.4 0.2 0.04"/>
+          </geometry>
+          <material name="gray"/>
+        </visual>
+        <collision>
+          <origin xyz="0 0 0"/>
+          <geometry>
+            <box size="0.4 0.2 0.04"/>
+          </geometry>
+        </collision>
+        <xacro:inertial_box mass="0.5" x="0.4" y="0.2" z="0.04"/>
+      </link>
+      <gazebo reference="base_link">
+        <material>Gazebo/Grey</material>
+      </gazebo>
+      <link name="FL">
+        <visual>
+          <origin xyz="0 0 0" rpy="${pi/2} 0 0" />
+          <geometry>
             <cylinder length="0.26" radius="0.015"/>
-         </geometry>
-         <material name="white"/>
-       </visual>
-     </link>
-     <link name="FR">
-       <visual>
-		 <origin xyz="0 0 0.04" rpy="${pi/2} 0 0" />
-         <geometry>
+          </geometry>
+          <material name="white"/>
+        </visual>
+        <collision>
+          <origin xyz="0 0 0" rpy="${pi/2} 0 0"/>
+          <geometry>
             <cylinder length="0.26" radius="0.015"/>
-         </geometry>
-         <material name="red"/>
-       </visual>
-     </link>
-     <link name="BL">
-       <visual>
-		 <origin xyz="0 0 0.04" rpy="${pi/2} 0 0" />
-         <geometry>
+          </geometry>
+        </collision>
+        <xacro:inertial_cylinder_y mass="0.05" l="0.26" r="0.015"/>
+      </link>
+      <gazebo reference="FL">
+        <material>Gazebo/White</material>
+      </gazebo>
+      <link name="FR">
+        <visual>
+          <origin xyz="0 0 0" rpy="${pi/2} 0 0" />
+          <geometry>
             <cylinder length="0.26" radius="0.015"/>
-         </geometry>
-         <material name="red"/>
-       </visual>
-     </link>
-     <link name="BR">
-       <visual>
-		 <origin xyz="0 0 0.04" rpy="${pi/2} 0 0" />
-         <geometry>
+          </geometry>
+          <material name="red"/>
+        </visual>
+        <collision>
+          <origin xyz="0 0 0" rpy="${pi/2} 0 0"/>
+          <geometry>
             <cylinder length="0.26" radius="0.015"/>
-         </geometry>
-         <material name="white"/>
-       </visual>
-     </link>
+          </geometry>
+        </collision>
+        <xacro:inertial_cylinder_y mass="0.05" l="0.26" r="0.015"/>
+      </link>
+      <gazebo reference="FR">
+        <material>Gazebo/Red</material>
+      </gazebo>
+      <link name="BL">
+        <visual>
+          <origin xyz="0 0 0" rpy="${pi/2} 0 0" />
+          <geometry>
+            <cylinder length="0.26" radius="0.015"/>
+          </geometry>
+          <material name="red"/>
+        </visual>
+        <collision>
+          <origin xyz="0 0 0" rpy="${pi/2} 0 0"/>
+          <geometry>
+            <cylinder length="0.26" radius="0.015"/>
+          </geometry>
+        </collision>
+        <xacro:inertial_cylinder_y mass="0.05" l="0.26" r="0.015"/>
+      </link>
+      <gazebo reference="BL">
+        <material>Gazebo/Red</material>
+      </gazebo>
+      <link name="BR">
+        <visual>
+          <origin xyz="0 0 0" rpy="${pi/2} 0 0" />
+          <geometry>
+            <cylinder length="0.26" radius="0.015"/>
+          </geometry>
+          <material name="white"/>
+        </visual>
+        <collision>
+          <origin xyz="0 0 0" rpy="${pi/2} 0 0"/>
+          <geometry>
+            <cylinder length="0.26" radius="0.015"/>
+          </geometry>
+        </collision>
+        <xacro:inertial_cylinder_y mass="0.05" l="0.26" r="0.015"/>
+      </link>
+      <gazebo reference="BR">
+        <material>Gazebo/White</material>
+      </gazebo>
      <joint name="base_to_FL" type="continuous">
        <parent link="base_link"/>
        <child link="FL"/>
-       <origin xyz="0.2 0.15 0" rpy="0 0 0" />
+       <origin xyz="0.2 0.15 0.04" rpy="0 0 0" />
        <axis xyz="0 0 1"/>
      </joint>
@@ -64,5 +115,5 @@
        <parent link="base_link"/>
        <child link="FR"/>
-       <origin xyz="0.2 -0.15 0" rpy="0 0 0" />
+       <origin xyz="0.2 -0.15 0.04" rpy="0 0 0" />
        <axis xyz="0 0 -1"/>
      </joint>
@@ -70,5 +121,5 @@
        <parent link="base_link"/>
        <child link="BL"/>
-       <origin xyz="-0.2 0.15 0" rpy="0 0 0" />
+       <origin xyz="-0.2 0.15 0.04" rpy="0 0 0" />
        <axis xyz="0 0 -1"/>
      </joint>
@@ -76,5 +127,5 @@
        <parent link="base_link"/>
        <child link="BR"/>
-       <origin xyz="-0.2 -0.15 0" rpy="0 0 0" />
+       <origin xyz="-0.2 -0.15 0.04" rpy="0 0 0" />
        <axis xyz="0 0 1"/>
      </joint>
